Commit message: complete gazebo_simulator

File: src/gazebo_simulator/urdf/diffbot.urdf.xacro (robot description, xacro)
@@ -1,4 +1,4 @@
 <?xml version='1.0'?>
-<robot name="skidbot" xmlns:xacro="http://www.ros.org/wiki/xacro">
+<robot name="diffbot" xmlns:xacro="http://www.ros.org/wiki/xacro">
   <xacro:include filename="$(find gazebo_simulator)/urdf/diffbot.gazebo" />
   <link name="robot_footprint"></link>
@@ -9,5 +9,5 @@
   </joint>
   <link name='chassis'>
-    <pose>0 0 0.1 0 0 0</pose>
+    <!-- <pose>0 0 0.1 0 0 0</pose> -->
     <inertial>
       <mass value="15.0"/>
@@ -136,5 +136,5 @@
       </geometry>
     </visual>
-    <collision name="camera_colision">
+    <collision name="camera_collision">
       <origin xyz="0 0 0" rpy="0 0 0" />
       <geometry>
@@ -155,5 +155,5 @@
       </geometry>
     </visual>
-    <collision name="hokuyo_colision">
+    <collision name="hokuyo_collision">
       <origin xyz="0 0 0" rpy="0 0 0" />
       <geometry>
@@ -200,5 +200,5 @@
     <axis xyz="0 1 0" rpy="0 0 0"/>
   </joint>
-  <gazebo reference="chassis">
+  <!-- <gazebo reference="chassis">
     <material>Gazebo/Green</material>
   </gazebo>
@@ -214,4 +214,4 @@
   <gazebo reference="hokuyo">
     <material>Gazebo/Black</material>
-  </gazebo>
+  </gazebo> -->
 </robot>
